Commit message: src

File: src/urdf_xacro/door_handle.urdf (robot description, URDF)
Before this commit: robot door_robot, 2 links, 1 joints
Links:
- link door_handle: geometry visual mesh filename=obj/handle_edited.obj rpy=0 0 0

File: src/urdf_xacro/door_handle.urdf.xacro (robot description, xacro)
@@ -26,5 +26,5 @@
                 <geometry>
                     <!-- <mesh filename="handle_edited.obj" rpy="0 0 0" /> -->
-                    <mesh filename="knob.obj" rpy="0 0 0" />
+                    <mesh filename="obj/knob_small.obj" rpy="0 0 0" />
                 </geometry>
                 <material name="wood">
@@ -56,5 +56,5 @@
                 <origin xyz="0 0 0" />
                 <geometry>
-                    <mesh filename="door2.obj" rpy="0 0 0" />
+                    <mesh filename="obj/door2.obj" rpy="0 0 0" />
                 </geometry>
                 <material name="wood">
