Commit message: README edited

File: src/urdf_xacro/door.urdf (robot description, URDF)
Before this commit: robot door_robot, 3 links, 2 joints
Links:
- link door_handle: geometry visual mesh filename=obj/handle_edited.obj rpy=0 0 0
- link door_plane: geometry visual mesh filename=obj/door2.obj rpy=0 0 0

File: src/urdf_xacro/door_handle.urdf.xacro (robot description, xacro)
@@ -3,5 +3,5 @@
     <xacro:arg name="parent" default="world"/>
     <xacro:property name="handle_pos_x" value="0.0"/>
-    <xacro:property name="handle_pos_y" value="0.25"/>
+    <xacro:property name="handle_pos_y" value="0.0"/>
     <xacro:property name="handle_pos_z" value="0.0"/>
     <xacro:macro name="door_robot" params="parent">

File: src/urdf_xacro/out.urdf (robot description, URDF)
Before this commit: robot door_robot, 3 links, 2 joints
Joints:
- joint handle_door: origin xyz=0.0 0.25 0.0 rpy=0 0 0 -> xyz=0.0 0.0 0.0 rpy=0 0 0

Commit message: usefull pdfs in docs

File: src/urdf_xacro/door.urdf (robot description, URDF)
Before this commit: robot door_robot, 3 links, 2 joints
Joints:
- removed joint door_handle_connect
- removed joint door_hinge
- added joint door_handle: type fixed, parent door_plane, child door_handle, origin xyz=0 0 0 rpy=0 0 0, axis 0 0 0, limit lower=0.0 upper=1.57
- added joint world_door: type fixed, parent world, child door_plane, origin xyz=0 0 1 rpy=0 0 0, axis 0 0 0, limit lower=0.0 upper=1.57

Commit message: minor changes in current urdf's

File: src/urdf_xacro/door.urdf (robot description, URDF)
Before this commit: robot door_robot, 3 links, 2 joints
Links:
- link door_handle: mass 2.6409912742551773 -> None
- link door_plane: mass 2.6409912742551773 -> None

File: src/urdf_xacro/door_handle.urdf (robot description, URDF)
Before this commit: robot door_robot, 2 links, 1 joints
Links:
- link door_handle: mass 2.6409912742551773 -> None
Joints:
- removed joint door_hinge
- added joint world_handle: type fixed, parent world, child door_handle, origin xyz=0 0 1 rpy=0 0 0, axis 0 0 0, limit lower=0.0 upper=1.57

File: src/urdf_xacro/door_handle.urdf.xacro (robot description, xacro)
@@ -17,9 +17,4 @@
         </joint>
         <link name="door_handle">
-            <inertial>
-                <origin xyz="0 0 0" />
-                <mass value="2.6409912742551773" />
-                <inertia ixx="0.0" ixy="0.0" ixz="0.0" iyy="0.0" iyz="0.0" izz="0.0" />
-            </inertial>
             <visual>
                 <origin xyz="0 0 0" />
@@ -32,5 +27,11 @@
                 </material>
             </visual>
-            <!--<collision>
+            <!--
+            <inertial>
+                <origin xyz="0 0 0" />
+                <mass value="2.6409912742551773" />
+                <inertia ixx="0.0" ixy="0.0" ixz="0.0" iyy="0.0" iyz="0.0" izz="0.0" />
+            </inertial>
+            <collision>
                 <origin xyz="-0.148404 0.486267 4.17233e-07" />
                 <geometry>
@@ -48,9 +49,4 @@
         </joint>
         <link name="door_plane">
-            <inertial>
-                <origin xyz="0 0 0" />
-                <mass value="2.6409912742551773" />
-                <inertia ixx="0.0" ixy="0.0" ixz="0.0" iyy="0.0" iyz="0.0" izz="0.0" />
-            </inertial>
             <visual>
                 <origin xyz="0 0 0" />
@@ -62,5 +58,11 @@
                 </material>
             </visual>
-            <!--<collision>
+            <!--
+            <inertial>
+                <origin xyz="0 0 0" />
+                <mass value="2.6409912742551773" />
+                <inertia ixx="0.0" ixy="0.0" ixz="0.0" iyy="0.0" iyz="0.0" izz="0.0" />
+            </inertial>
+            <collision>
                 <origin xyz="-0.148404 0.486267 4.17233e-07" />
                 <geometry>

File: src/urdf_xacro/out.urdf (robot description, URDF)
Before this commit: robot door_robot, 3 links, 2 joints
Links:
- link door_handle: mass 2.6409912742551773 -> None
- link door_plane: mass 2.6409912742551773 -> None
