Commit message: Fixes

File: src/urdf_xacro/handle.xacro (robot description, xacro)
@@ -5,5 +5,5 @@
     <xacro:property name="handle_pos_y" value="0.0"/>
     <xacro:property name="handle_pos_z" value="0.0"/>
-    <xacro:macro name="door_handle" params="parent">
+    <xacro:macro name="door_handle" params="handle_file">
         <link name="world"/>
         <joint name="handle_door" type="fixed">
@@ -41,4 +41,3 @@
         </link>
     </xacro:macro>
-    <xacro:door_handle parent="$(arg handle_file)"/>
 </robot>

File: src/urdf_xacro/plane.xacro (robot description, xacro)
@@ -5,5 +5,5 @@
     <xacro:arg name="size_y" default="0.0"/>
     <xacro:arg name="size_z" default="0.0"/>
-    <xacro:macro name="door_plane" params="plane_file">
+    <xacro:macro name="door_plane" params="plane_file" "size_x" "size_y" "size_z">
         <link name="world"/>
         <joint name="door_world" type="fixed">
@@ -39,4 +39,3 @@
         </link>
     </xacro:macro>
-    <xacro:door_plane plane_file="$(arg plane_file)" size_x="$(size_x)" size_y="$(size_y)" size_z="$(size_z)"/>
 </robot>

Commit message: Added parent parameter for handle macro

File: src/urdf_xacro/handle.xacro (robot description, xacro)
@@ -2,13 +2,14 @@
 <robot name="door_handle" xmlns:xacro="http://www.ros.org/wiki/xacro">
     <xacro:arg name="handle_file" default=""/>
+    <xacro:arg name="parent" default="world"/>
     <xacro:property name="handle_pos_x" value="0.0"/>
     <xacro:property name="handle_pos_y" value="0.0"/>
     <xacro:property name="handle_pos_z" value="0.0"/>
     <xacro:macro name="door_handle" params="handle_file">
-        <link name="world"/>
+        <link name="${parent}"/>
         <joint name="handle_door" type="fixed">
             <!-- Hier xyz für door zu handle offset -->
             <origin xyz="${handle_pos_x} ${handle_pos_y} ${handle_pos_z}" rpy="0 0 0" />
-            <parent link="world" />
+            <parent link="${parent}" />
             <child link="door_handle" />
             <axis xyz="0 0 0" />
