Commit message: Fixed params

File: src/urdf_xacro/door_handle.urdf.xacro (robot description, xacro)
@@ -5,5 +5,5 @@
     <xacro:property name="handle_pos_y" value="0.0"/>
     <xacro:property name="handle_pos_z" value="0.0"/>
-    <xacro:macro name="door_robot" params="parent">
+    <xacro:macro name="door_robot" params="parent handle_pos_x handle_pos_y handle_pos_z">
         <link name="${parent}"/>
         <joint name="handle_door" type="fixed">

File: src/urdf_xacro/handle.xacro (robot description, xacro)
@@ -6,5 +6,5 @@
     <xacro:property name="handle_pos_y" value="0.0"/>
     <xacro:property name="handle_pos_z" value="0.0"/>
-    <xacro:macro name="door_handle" params="handle_file">
+    <xacro:macro name="door_handle" params="handle_file parent handle_pos_x handle_pos_y handle_pos_z">
         <link name="${parent}"/>
         <joint name="handle_door" type="fixed">
