Commit message: Added door scale as parameter

File: src/urdf_xacro/plane.xacro (robot description, xacro)
@@ -19,5 +19,5 @@
                 <origin xyz="0 0 0" />
                 <geometry>
-                    <mesh filename="${plane_file}" rpy="0 0 0" />
+                    <mesh filename="${plane_file}" rpy="0 0 0" scale="${size_x} ${size_y} ${size_z}" />
                 </geometry>
                 <material name="wood">
@@ -39,4 +39,4 @@
         </link>
     </xacro:macro>
-    <xacro:door_plane plane_file="$(arg plane_file)"/>
+    <xacro:door_plane plane_file="$(arg plane_file)" size_x="$(size_x)" size_y="$(size_y)" size_z="$(size_z)"/>
 </robot>

Commit message: Fixed plane params

File: src/urdf_xacro/plane.xacro (robot description, xacro)
@@ -5,5 +5,5 @@
     <xacro:arg name="size_y" default="0.0"/>
     <xacro:arg name="size_z" default="0.0"/>
-    <xacro:macro name="door_plane" params="plane_file" "size_x" "size_y" "size_z">
+    <xacro:macro name="door_plane" params="plane_file size_x size_y size_z">
         <link name="world"/>
         <joint name="door_world" type="fixed">

Commit message: Added xacro_processor

File: src/urdf_xacro/plane.xacro (robot description, xacro)
@@ -2,13 +2,14 @@
 <robot name="door_plane" xmlns:xacro="http://www.ros.org/wiki/xacro">
     <xacro:arg name="plane_file" default=""/>
+    <xacro:arg name="parent" default="world"/>
     <xacro:arg name="size_x" default="0.0"/>
     <xacro:arg name="size_y" default="0.0"/>
     <xacro:arg name="size_z" default="0.0"/>
-    <xacro:macro name="door_plane" params="plane_file size_x size_y size_z">
-        <link name="world"/>
+    <xacro:macro name="door_plane" params="plane_file parent size_x size_y size_z">
+        <link name="${parent}"/>
         <joint name="door_world" type="fixed">
             <origin xyz="0 0 1" rpy="0 0 0" />
-            <parent link="world" />
-            <child link="door_plane" />
+            <parent link="${parent}" />
+            <child link="plane" />
             <axis xyz="0 0 0" />
             <dynamics friction="0.4960139088111456" />
@@ -39,3 +40,4 @@
         </link>
     </xacro:macro>
+    <xacro:door_plane plane_file="$(arg plane_file)" parent="$(arg parent)" size_x="$(arg size_x)" size_y="$(arg size_y)" size_z="$(arg size_z)"/>
 </robot>
