Commit message: Fix xacro

File: scripts/handle.xacro (robot description, xacro)
@@ -1,13 +1,14 @@
 <?xml version="1.0" encoding="utf-8"?>
 <robot name="door_handle" xmlns:xacro="http://www.ros.org/wiki/xacro">
-    <xacro:arg name="mesh_file" default="handle_edited.obj"/>
+    <xacro:property name="mesh_file" value="handle_edited.obj"/>
     <xacro:arg name="parent" default="world"/>
-    <xacro:property name="handle_pos_x" value="0.0"/>
-    <xacro:property name="handle_pos_y" value="0.0"/>
-    <xacro:property name="handle_pos_z" value="0.0"/>
-    <xacro:property name="handle_ori_r" value="0.0"/>
-    <xacro:property name="handle_ori_p" value="0.0"/>
-    <xacro:property name="handle_ori_y" value="0.0"/>
-    <xacro:macro name="door_handle" params="mesh_file parent handle_pos_x handle_pos_y handle_pos_z handle_ori_r handle_ori_p handle_ori_y">
+    <xacro:property name="mesh_file" value="handle_edited.obj"/>
+    <xacro:arg name="handle_pos_x" default="0.0"/>
+    <xacro:arg name="handle_pos_y" default="0.0"/>
+    <xacro:arg name="handle_pos_z" default="0.0"/>
+    <xacro:arg name="handle_ori_r" default="0.0"/>
+    <xacro:arg name="handle_ori_p" default="0.0"/>
+    <xacro:arg name="handle_ori_y" default="0.0"/>
+    <xacro:macro name="door_handle" params="parent handle_pos_x handle_pos_y handle_pos_z handle_ori_r handle_ori_p handle_ori_y">
         <link name="${parent}"/>
         <joint name="handle_door" type="fixed">

File: scripts/plane.xacro (robot description, xacro)
@@ -1,10 +1,10 @@
 <?xml version="1.0" encoding="utf-8"?>
 <robot name="door_plane" xmlns:xacro="http://www.ros.org/wiki/xacro">
-    <xacro:arg name="mesh_file" default="door2.obj"/>
     <xacro:arg name="parent" default="world"/>
-    <xacro:property name="size_x" default="0.0"/>
-    <xacro:property name="size_y" default="0.0"/>
-    <xacro:property name="size_z" default="0.0"/>
-    <xacro:macro name="door_plane" params="mesh_file parent">
+    <xacro:property name="mesh_file" value="door2.obj"/>
+    <xacro:property name="size_x" value="1.0"/>
+    <xacro:property name="size_y" value="1.0"/>
+    <xacro:property name="size_z" value="1.0"/>
+    <xacro:macro name="door_plane" params="parent">
         <link name="${parent}"/>
         <joint name="door_world" type="fixed">
@@ -40,4 +40,3 @@
         </link>
     </xacro:macro>
-    <xacro:door_plane mesh_file="$(arg mesh_file)" parent="$(arg parent)"/>
 </robot>

File: src/urdf_xacro/complete_door.xacro (robot description, xacro)
@@ -1,6 +1,6 @@
 <?xml version="1.0" encoding="utf-8"?>
 <robot name="complete door" xmlns:xacro="http://www.ros.org/wiki/xacro">
-    <xacro:property name="plane_xacro" default=""/>
-    <xacro:property name="handle_xacro" default=""/>
+    <xacro:property name="plane_xacro" default="plane.xacro"/>
+    <xacro:property name="handle_xacro" default="handle.xacro"/>
     <xacro:property name="handle_pos_x" value="0.0"/>
     <xacro:property name="handle_pos_y" value="0.0"/>
@@ -9,11 +9,8 @@
     <xacro:property name="handle_ori_p" value="0.0"/>
     <xacro:property name="handle_ori_y" value="0.0"/>
-    <xacro:property name="size_x" default="0.0"/>
-    <xacro:property name="size_y" default="0.0"/>
-    <xacro:property name="size_z" default="0.0"/>
-    <xacro::include filename=${plane_xacro}
+    <xacro:include filename="${plane_xacro}"/>
     <xacro:door_plane parent="world"/>
-    <xacro:include filename=${handle_xacro}
+    <xacro:include filename="${handle_xacro}"/>
     <xacro:door_handle parent="door_plane" handle_pos_x="${handle_pos_x}" handle_pos_y="${handle_pos_y}"
-    handle_pos_z="${handle_pos_z}" handle_ori_r="${handle_ori_r}" handle_ori_p="${handle_ori_p}" handle_ori_y="${handle_ori_y}"
+    handle_pos_z="${handle_pos_z}" handle_ori_r="${handle_ori_r}" handle_ori_p="${handle_ori_p}" handle_ori_y="${handle_ori_y}"/>
 </robot>
