Commit message: Added complete door

File: data/objs/pieces/doors/plane.xacro (robot description, xacro)
@@ -3,8 +3,8 @@
     <xacro:arg name="plane_file" default=""/>
     <xacro:arg name="parent" default="world"/>
-    <xacro:arg name="size_x" default="0.0"/>
-    <xacro:arg name="size_y" default="0.0"/>
-    <xacro:arg name="size_z" default="0.0"/>
-    <xacro:macro name="door_plane" params="plane_file parent size_x size_y size_z">
+    <xacro:property name="size_x" default="0.0"/>
+    <xacro:property name="size_y" default="0.0"/>
+    <xacro:property name="size_z" default="0.0"/>
+    <xacro:macro name="door_plane" params="plane_file parent ">
         <link name="${parent}"/>
         <joint name="door_world" type="fixed">
@@ -40,4 +40,4 @@
         </link>
     </xacro:macro>
-    <xacro:door_plane plane_file="$(arg plane_file)" parent="$(arg parent)" size_x="$(arg size_x)" size_y="$(arg size_y)" size_z="$(arg size_z)"/>
+    <xacro:door_plane plane_file="$(arg plane_file)" parent="$(arg parent)"/>
 </robot>

File: src/urdf_xacro/complete_door.xacro (robot description, xacro)
@@ -5,79 +5,15 @@
     <xacro:arg name="handle_pos_x" value="0.0"/>
     <xacro:arg name="handle_pos_y" value="0.0"/>
-    <xacro:arg name="handle_pos_z" value="0.0"/>
+    <xacro:arg name="handle_pos_z" value="1.0"/>
+    <xacro:arg name="handle_ori_r" value="0.0"/>
+    <xacro:arg name="handle_ori_p" value="0.0"/>
+    <xacro:arg name="handle_ori_y" value="0.0"/>
     <xacro:property name="size_x" default="0.0"/>
     <xacro:property name="size_y" default="0.0"/>
     <xacro:property name="size_z" default="0.0"/>
-    <xacro:::include filename=${plane_file}
-    <xacro:::include filename=${handle_file}
-    <xacro:macro name="complete door" params="plane_file" "handle_file" "handle_pos_x" "handle_pos_y" "handle_pos_z">
-        <link name="world"/>
-        <xacro::door_handle params=${handle_file}/>
-        <xacro::door_handle params=${plane_file} ${size_x} ${size_y} ${size_z}/>
-        <joint name="handle_door" type="fixed">
-            <!-- Hier xyz für door zu handle offset -->
-            <origin xyz="${handle_pos_x} ${handle_pos_y} ${handle_pos_z}" rpy="0 0 0" />
-            <parent link="door_plane" />
-            <child link="door_handle" />
-            <axis xyz="0 0 0" />
-            <dynamics friction="0.4960139088111456" />
-            <limit lower="0.0" upper="1.57"/>
-        </joint>
-        <link name="door_handle">
-            <visual>
-                <origin xyz="0 0 0" />
-                <geometry>
-                    <!-- <mesh filename="handle_edited.obj" rpy="0 0 0" /> -->
-                    <mesh filename="obj/knob_small.obj" rpy="0 0 0" />
-                </geometry>
-                <material name="wood">
-                <color rgba ="1 1 1 1"/>
-                </material>
-            </visual>
-            <!--
-            <inertial>
-                <origin xyz="0 0 0" />
-                <mass value="2.6409912742551773" />
-                <inertia ixx="0.0" ixy="0.0" ixz="0.0" iyy="0.0" iyz="0.0" izz="0.0" />
-            </inertial>
-            <collision>
-                <origin xyz="-0.148404 0.486267 4.17233e-07" />
-                <geometry>
-                    <mesh filename="handle_edited.obj" rpy="0 0 0" />
-                </geometry>
-            </collision>-->
-        </link>
-        <joint name="door_world" type="fixed">
-            <origin xyz="0 0 1" rpy="0 0 0" />
-            <parent link="${parent}" />
-            <child link="door_plane" />
-            <axis xyz="0 0 0" />
-            <dynamics friction="0.4960139088111456" />
-            <limit lower="0.0" upper="1.57"/>
-        </joint>
-        <link name="door_plane">
-            <visual>
-                <origin xyz="0 0 0" />
-                <geometry>
-                    <mesh filename="obj/door2.obj" rpy="0 0 0" />
-                </geometry>
-                <material name="wood">
-                <color rgba ="1 1 1 1"/>
-                </material>
-            </visual>
-            <!--
-            <inertial>
-                <origin xyz="0 0 0" />
-                <mass value="2.6409912742551773" />
-                <inertia ixx="0.0" ixy="0.0" ixz="0.0" iyy="0.0" iyz="0.0" izz="0.0" />
-            </inertial>
-            <collision>
-                <origin xyz="-0.148404 0.486267 4.17233e-07" />
-                <geometry>
-                    <mesh filename="door2.obj" rpy="0 0 0" />
-                </geometry>
-            </collision>-->
-        </link>
-    </xacro:macro>
-    <xacro:door_robot parent="$(arg parent)"/>
+    <xacro::include filename=${plane_file}
+    <xacro:door_plane plane_file="${plane_file}" parent="world"/>
+    <xacro:include filename=${handle_file}
+    <xacro:door_handle handle_file="${handle_file}" parent="door_plane" handle_pos_x="${handle_pos_x}" handle_pos_y="${handle_pos_y}"
+    handle_pos_z="${handle_pos_z}" handle_ori_r="${handle_ori_r}" handle_ori_p="${handle_ori_p}" handle_ori_y="${handle_ori_y}"
 </robot>

Commit message: Fixed plane

File: data/objs/pieces/doors/plane.xacro (robot description, xacro)
@@ -6,5 +6,5 @@
     <xacro:property name="size_y" default="0.0"/>
     <xacro:property name="size_z" default="0.0"/>
-    <xacro:macro name="door_plane" params="plane_file parent ">
+    <xacro:macro name="door_plane" params="plane_file parent">
         <link name="${parent}"/>
         <joint name="door_world" type="fixed">

Commit message: Changed mesh and xacro filename property

File: data/objs/pieces/doors/plane.xacro (robot description, xacro)
@@ -1,10 +1,10 @@
 <?xml version="1.0" encoding="utf-8"?>
 <robot name="door_plane" xmlns:xacro="http://www.ros.org/wiki/xacro">
-    <xacro:arg name="plane_file" default=""/>
+    <xacro:arg name="mesh_file" default=""/>
     <xacro:arg name="parent" default="world"/>
     <xacro:property name="size_x" default="0.0"/>
     <xacro:property name="size_y" default="0.0"/>
     <xacro:property name="size_z" default="0.0"/>
-    <xacro:macro name="door_plane" params="plane_file parent">
+    <xacro:macro name="door_plane" params="mesh_file parent">
         <link name="${parent}"/>
         <joint name="door_world" type="fixed">
@@ -20,5 +20,5 @@
                 <origin xyz="0 0 0" />
                 <geometry>
-                    <mesh filename="${plane_file}" rpy="0 0 0" scale="${size_x} ${size_y} ${size_z}" />
+                    <mesh filename="${mesh_file}" rpy="0 0 0" scale="${size_x} ${size_y} ${size_z}" />
                 </geometry>
                 <material name="wood">
@@ -40,4 +40,4 @@
         </link>
     </xacro:macro>
-    <xacro:door_plane plane_file="$(arg plane_file)" parent="$(arg parent)"/>
+    <xacro:door_plane plane_file="$(arg mesh_file)" parent="$(arg parent)"/>
 </robot>

File: data/objs/pieces/handles/handle.xacro (robot description, xacro)
@@ -1,5 +1,5 @@
 <?xml version="1.0" encoding="utf-8"?>
 <robot name="door_handle" xmlns:xacro="http://www.ros.org/wiki/xacro">
-    <xacro:arg name="handle_file" default=""/>
+    <xacro:arg name="mesh_file" default=""/>
     <xacro:arg name="parent" default="world"/>
     <xacro:property name="handle_pos_x" value="0.0"/>
@@ -9,5 +9,5 @@
     <xacro:property name="handle_ori_p" value="0.0"/>
     <xacro:property name="handle_ori_y" value="0.0"/>
-    <xacro:macro name="door_handle" params="handle_file parent handle_pos_x handle_pos_y handle_pos_z handle_ori_r handle_ori_p handle_ori_y">
+    <xacro:macro name="door_handle" params="mesh_file parent handle_pos_x handle_pos_y handle_pos_z handle_ori_r handle_ori_p handle_ori_y">
         <link name="${parent}"/>
         <joint name="handle_door" type="fixed">
@@ -25,5 +25,5 @@
                 <geometry>
                     <!-- <mesh filename="handle_edited.obj" rpy="0 0 0" /> -->
-                    <mesh filename="${handle_file}" rpy="0 0 0" />
+                    <mesh filename="${mesh_file}" rpy="0 0 0" />
                 </geometry>
                 <material name="wood">

File: src/urdf_xacro/complete_door.xacro (robot description, xacro)
@@ -1,6 +1,6 @@
 <?xml version="1.0" encoding="utf-8"?>
 <robot name="complete door" xmlns:xacro="http://www.ros.org/wiki/xacro">
-    <xacro:property name="plane_file" default=""/>
-    <xacro:property name="handle_file" default=""/>
+    <xacro:property name="plane_xacro" default=""/>
+    <xacro:property name="handle_xacro" default=""/>
     <xacro:property name="handle_pos_x" value="0.0"/>
     <xacro:property name="handle_pos_y" value="0.0"/>
@@ -12,8 +12,8 @@
     <xacro:property name="size_y" default="0.0"/>
     <xacro:property name="size_z" default="0.0"/>
-    <xacro::include filename=${plane_file}
-    <xacro:door_plane plane_file="${plane_file}" parent="world"/>
-    <xacro:include filename=${handle_file}
-    <xacro:door_handle handle_file="${handle_file}" parent="door_plane" handle_pos_x="${handle_pos_x}" handle_pos_y="${handle_pos_y}"
+    <xacro::include filename=${plane_xacro}
+    <xacro:door_plane parent="world"/>
+    <xacro:include filename=${handle_xacro}
+    <xacro:door_handle parent="door_plane" handle_pos_x="${handle_pos_x}" handle_pos_y="${handle_pos_y}"
     handle_pos_z="${handle_pos_z}" handle_ori_r="${handle_ori_r}" handle_ori_p="${handle_ori_p}" handle_ori_y="${handle_ori_y}"
 </robot>

Commit message: Fixed xacros

File: data/objs/pieces/doors/plane.xacro (robot description, xacro)
@@ -1,24 +1,24 @@
 <?xml version="1.0" encoding="utf-8"?>
 <robot name="door_plane" xmlns:xacro="http://www.ros.org/wiki/xacro">
-    <xacro:arg name="mesh_file" default="door2.obj"/>
     <xacro:arg name="parent" default="world"/>
-    <xacro:property name="size_x" default="0.0"/>
-    <xacro:property name="size_y" default="0.0"/>
-    <xacro:property name="size_z" default="0.0"/>
-    <xacro:macro name="door_plane" params="mesh_file parent">
+    <xacro:property name="door_mesh_file" value="door2.obj"/>
+    <xacro:property name="size_x" value="1.0"/>
+    <xacro:property name="size_y" value="1.0"/>
+    <xacro:property name="size_z" value="1.0"/>
+    <xacro:macro name="door_plane" params="parent">
         <link name="${parent}"/>
         <joint name="door_world" type="fixed">
             <origin xyz="0 0 1" rpy="0 0 0" />
             <parent link="${parent}" />
-            <child link="plane" />
+            <child link="door_plane" />
             <axis xyz="0 0 0" />
             <dynamics friction="0.4960139088111456" />
             <limit lower="0.0" upper="1.57"/>
         </joint>
-        <link name="plane">
+        <link name="door_plane">
             <visual>
                 <origin xyz="0 0 0" />
                 <geometry>
-                    <mesh filename="${mesh_file}" rpy="0 0 0" scale="${size_x} ${size_y} ${size_z}" />
+                    <mesh filename="${door_mesh_file}" rpy="0 0 0" scale="${size_x} ${size_y} ${size_z}" />
                 </geometry>
                 <material name="wood">
@@ -40,4 +40,3 @@
         </link>
     </xacro:macro>
-    <xacro:door_plane mesh_file="$(arg mesh_file)" parent="$(arg parent)"/>
 </robot>

File: data/objs/pieces/handles/handle.xacro (robot description, xacro)
@@ -1,18 +1,16 @@
 <?xml version="1.0" encoding="utf-8"?>
 <robot name="door_handle" xmlns:xacro="http://www.ros.org/wiki/xacro">
-    <xacro:arg name="mesh_file" default="handle_edited.obj"/>
-    <xacro:arg name="parent" default="world"/>
-    <xacro:property name="handle_pos_x" value="0.0"/>
-    <xacro:property name="handle_pos_y" value="0.0"/>
-    <xacro:property name="handle_pos_z" value="0.0"/>
-    <xacro:property name="handle_ori_r" value="0.0"/>
-    <xacro:property name="handle_ori_p" value="0.0"/>
-    <xacro:property name="handle_ori_y" value="0.0"/>
-    <xacro:macro name="door_handle" params="mesh_file parent handle_pos_x handle_pos_y handle_pos_z handle_ori_r handle_ori_p handle_ori_y">
-        <link name="${parent}"/>
+    <xacro:property name="handle_mesh_file" value="handle_edited.obj"/>
+    <xacro:arg name="handle_pos_x" default="0.0"/>
+    <xacro:arg name="handle_pos_y" default="0.0"/>
+    <xacro:arg name="handle_pos_z" default="0.0"/>
+    <xacro:arg name="handle_ori_r" default="0.0"/>
+    <xacro:arg name="handle_ori_p" default="0.0"/>
+    <xacro:arg name="handle_ori_y" default="0.0"/>
+    <xacro:macro name="door_handle" params="handle_pos_x handle_pos_y handle_pos_z handle_ori_r handle_ori_p handle_ori_y">
         <joint name="handle_door" type="fixed">
             <!-- Hier xyz für door zu handle offset -->
             <origin xyz="${handle_pos_x} ${handle_pos_y} ${handle_pos_z}" rpy="${handle_ori_r} ${handle_ori_p} ${handle_ori_y}" />
-            <parent link="${parent}" />
+            <parent link="door_plane" />
             <child link="door_handle" />
             <axis xyz="0 0 0" />
@@ -25,5 +23,5 @@
                 <geometry>
                     <!-- <mesh filename="handle_edited.obj" rpy="0 0 0" /> -->
-                    <mesh filename="${mesh_file}" rpy="0 0 0" />
+                    <mesh filename="${handle_mesh_file}" rpy="0 0 0" />
                 </geometry>
                 <material name="wood">

File: src/complete_door.xacro (robot description, xacro)
@@ -4,6 +4,6 @@
     <xacro:property name="handle_xacro" value="handle.xacro"/>
     <xacro:property name="handle_pos_x" value="0.0"/>
-    <xacro:property name="handle_pos_y" value="0.0"/>
-    <xacro:property name="handle_pos_z" value="1.0"/>
+    <xacro:property name="handle_pos_y" value="0.3"/>
+    <xacro:property name="handle_pos_z" value="0.0"/>
     <xacro:property name="handle_ori_r" value="0.0"/>
     <xacro:property name="handle_ori_p" value="0.0"/>
@@ -11,15 +11,6 @@
     <xacro:include filename="plane.xacro"/>
     <xacro:door_plane parent="world"/>
-    <link name="handle_connect"/>
-        <joint name="handle_joint" type="fixed">
-            <origin xyz="0 0 0" rpy="0 0 0" />
-            <parent link="door_plane" />
-            <child link="handle_connect" />
-            <axis xyz="0 0 0" />
-            <dynamics friction="0.4960139088111456" />
-            <limit lower="0.0" upper="1.57"/>
-        </joint>
-        <xacro:include filename="handle.xacro"/>
-    <xacro:door_handle parent="handle_connect" handle_pos_x="${handle_pos_x}" handle_pos_y="${handle_pos_y}"
+    <xacro:include filename="handle.xacro"/>
+    <xacro:door_handle handle_pos_x="${handle_pos_x}" handle_pos_y="${handle_pos_y}"
     handle_pos_z="${handle_pos_z}" handle_ori_r="${handle_ori_r}" handle_ori_p="${handle_ori_p}" handle_ori_y="${handle_ori_y}"/>
 </robot>

Commit message: Removed deprecated code

File: data/objs/pieces/doors/plane.xacro (robot description, xacro)
@@ -26,16 +26,4 @@
                 </material>
             </visual>
-            <!--
-            <inertial>
-                <origin xyz="0 0 0" />
-                <mass value="2.6409912742551773" />
-                <inertia ixx="0.0" ixy="0.0" ixz="0.0" iyy="0.0" iyz="0.0" izz="0.0" />
-            </inertial>
-            <collision>
-                <origin xyz="-0.148404 0.486267 4.17233e-07" />
-                <geometry>
-                    <mesh filename="door2.obj" rpy="0 0 0" />
-                </geometry>
-            </collision>-->
         </link>
     </xacro:macro>

File: data/objs/pieces/handles/handle.xacro (robot description, xacro)
@@ -10,5 +10,4 @@
     <xacro:macro name="door_handle" params="handle_pos_x handle_pos_y handle_pos_z handle_ori_r handle_ori_p handle_ori_y">
         <joint name="handle_door" type="fixed">
-            <!-- Hier xyz für door zu handle offset -->
             <origin xyz="${handle_pos_x} ${handle_pos_y} ${handle_pos_z}" rpy="${handle_ori_r} ${handle_ori_p} ${handle_ori_y}" />
             <parent link="door_plane" />
@@ -22,5 +21,4 @@
                 <origin xyz="0 0 0" />
                 <geometry>
-                    <!-- <mesh filename="handle_edited.obj" rpy="0 0 0" /> -->
                     <mesh filename="${handle_mesh_file}" rpy="0 0 0" />
                 </geometry>

File: scripts/complete_door.xacro (robot description, xacro)
@@ -9,7 +9,7 @@
     <xacro:property name="handle_ori_p" value="0.0"/>
     <xacro:property name="handle_ori_y" value="0.0"/>
-    <xacro:include filename="plane.xacro"/>
+    <xacro:include filename="${plane_xacro}"/>
     <xacro:door_plane parent="world"/>
-    <xacro:include filename="handle.xacro"/>
+    <xacro:include filename="${handle_xacro}"/>
     <xacro:door_handle handle_pos_x="${handle_pos_x}" handle_pos_y="${handle_pos_y}"
     handle_pos_z="${handle_pos_z}" handle_ori_r="${handle_ori_r}" handle_ori_p="${handle_ori_p}" handle_ori_y="${handle_ori_y}"/>

Commit message: data generation process

File: data/objs/pieces/doors/plane.xacro (robot description, xacro)
@@ -1,4 +1,5 @@
 <?xml version="1.0" encoding="utf-8"?>
 <robot name="door_plane" xmlns:xacro="http://www.ros.org/wiki/xacro">
+    <!--
     <xacro:arg name="parent" default="world"/>
     <xacro:property name="door_mesh_file" value="door2.obj"/>
@@ -6,8 +7,9 @@
     <xacro:property name="size_y" value="1.0"/>
     <xacro:property name="size_z" value="1.0"/>
+    -->
     <xacro:macro name="door_plane" params="parent">
         <link name="${parent}"/>
         <joint name="door_world" type="fixed">
-            <origin xyz="0 0 1" rpy="0 0 0" />
+            <origin xyz="0 0 ${z_origin}" rpy="0 0 0" />
             <parent link="${parent}" />
             <child link="door_plane" />

File: data/objs/pieces/handles/handle.xacro (robot description, xacro)
@@ -1,4 +1,5 @@
 <?xml version="1.0" encoding="utf-8"?>
 <robot name="door_handle" xmlns:xacro="http://www.ros.org/wiki/xacro">
+    <!--
     <xacro:property name="handle_mesh_file" value="handle_edited.obj"/>
     <xacro:arg name="handle_pos_x" default="0.0"/>
@@ -8,4 +9,5 @@
     <xacro:arg name="handle_ori_p" default="0.0"/>
     <xacro:arg name="handle_ori_y" default="0.0"/>
+    -->
     <xacro:macro name="door_handle" params="handle_pos_x handle_pos_y handle_pos_z handle_ori_r handle_ori_p handle_ori_y">
         <joint name="handle_door" type="fixed">

Commit message: Added collision to xacros

File: data/objs/pieces/doors/plane.xacro (robot description, xacro)
@@ -24,8 +24,11 @@
                     <mesh filename="${door_mesh_file}" rpy="0 0 0" scale="${size_x} ${size_y} ${size_z}" />
                 </geometry>
-                <material name="wood">
-                <color rgba ="1 1 1 1"/>
-                </material>
             </visual>
+            <collision>
+                <origin xyz="0 0 0" />
+                <geometry>
+                    <mesh filename="${door_mesh_file}" rpy="0 0 0" scale="${size_x} ${size_y} ${size_z}" />
+                </geometry>
+            </collision>
         </link>
     </xacro:macro>

File: data/objs/pieces/handles/handle.xacro (robot description, xacro)
@@ -25,20 +25,11 @@
                     <mesh filename="${handle_mesh_file}" rpy="0 0 0" />
                 </geometry>
-                <material name="wood">
-                <color rgba ="1 1 1 1"/>
-                </material>
             </visual>
-            <!--
-            <inertial>
+            <collision>
                 <origin xyz="0 0 0" />
-                <mass value="2.6409912742551773" />
-                <inertia ixx="0.0" ixy="0.0" ixz="0.0" iyy="0.0" iyz="0.0" izz="0.0" />
-            </inertial>
-            <collision>
-                <origin xyz="-0.148404 0.486267 4.17233e-07" />
                 <geometry>
-                    <mesh filename="handle_edited.obj" rpy="0 0 0" />
+                    <mesh filename="${handle_mesh_file}" rpy="0 0 0" />
                 </geometry>
-            </collision>-->
+            </collision>
         </link>
     </xacro:macro>
