Commit message: Added handle orientation parameter

File: data/objs/pieces/handles/handle.xacro (robot description, xacro)
@@ -6,9 +6,12 @@
     <xacro:property name="handle_pos_y" value="0.0"/>
     <xacro:property name="handle_pos_z" value="0.0"/>
-    <xacro:macro name="door_handle" params="handle_file parent handle_pos_x handle_pos_y handle_pos_z">
+    <xacro:property name="handle_ori_r" value="0.0"/>
+    <xacro:property name="handle_ori_p" value="0.0"/>
+    <xacro:property name="handle_ori_y" value="0.0"/>
+    <xacro:macro name="door_handle" params="handle_file parent handle_pos_x handle_pos_y handle_pos_z handle_ori_r handle_ori_p handle_ori_y">
         <link name="${parent}"/>
         <joint name="handle_door" type="fixed">
             <!-- Hier xyz für door zu handle offset -->
-            <origin xyz="${handle_pos_x} ${handle_pos_y} ${handle_pos_z}" rpy="0 0 0" />
+            <origin xyz="${handle_pos_x} ${handle_pos_y} ${handle_pos_z}" rpy="${handle_ori_r} ${handle_ori_p} ${handle_ori_y}" />
             <parent link="${parent}" />
             <child link="door_handle" />

Commit message: Changed xacro structure

File: data/objs/pieces/handles/handle.xacro (robot description, xacro)
@@ -2,11 +2,11 @@
 <robot name="door_handle" xmlns:xacro="http://www.ros.org/wiki/xacro">
     <xacro:property name="handle_mesh_file" value="handle_edited.obj"/>
-    <xacro:arg name="handle_pos_x" default="0.0"/>
-    <xacro:arg name="handle_pos_y" default="0.0"/>
-    <xacro:arg name="handle_pos_z" default="0.0"/>
-    <xacro:arg name="handle_ori_r" default="0.0"/>
-    <xacro:arg name="handle_ori_p" default="0.0"/>
-    <xacro:arg name="handle_ori_y" default="0.0"/>
-    <xacro:macro name="door_handle" params="handle_pos_x handle_pos_y handle_pos_z handle_ori_r handle_ori_p handle_ori_y">
+    <xacro:property name="handle_pos_x" value="0.0"/>
+    <xacro:property name="handle_pos_y" value="0.3"/>
+    <xacro:property name="handle_pos_z" value="0.0"/>
+    <xacro:property name="handle_ori_r" value="0.0"/>
+    <xacro:property name="handle_ori_p" value="0.0"/>
+    <xacro:property name="handle_ori_y" value="0.0"/>
+    <xacro:macro name="door_handle" params="">
         <joint name="handle_door" type="fixed">
             <!-- Hier xyz für door zu handle offset -->

File: scripts/complete_door.xacro (robot description, xacro)
@@ -3,14 +3,7 @@
     <xacro:property name="plane_xacro" value="plane.xacro"/>
     <xacro:property name="handle_xacro" value="handle.xacro"/>
-    <xacro:arg name="handle_pos_x" default="0.0"/>
-    <xacro:arg name="handle_pos_y" default="0.3"/>
-    <xacro:arg name="handle_pos_z" default="0.0"/>
-    <xacro:arg name="handle_ori_r" default="0.0"/>
-    <xacro:arg name="handle_ori_p" default="0.0"/>
-    <xacro:arg name="handle_ori_y" default="0.0"/>
     <xacro:include filename="plane.xacro"/>
     <xacro:door_plane parent="world"/>
     <xacro:include filename="handle.xacro"/>
-    <xacro:door_handle handle_pos_x="${handle_pos_x}" handle_pos_y="${handle_pos_y}"
-    handle_pos_z="${handle_pos_z}" handle_ori_r="${handle_ori_r}" handle_ori_p="${handle_ori_p}" handle_ori_y="${handle_ori_y}"/>
+    <xacro:door_handle/>
 </robot>

Commit message: Handle pose can be arg

File: data/objs/pieces/handles/handle.xacro (robot description, xacro)
@@ -2,11 +2,11 @@
 <robot name="door_handle" xmlns:xacro="http://www.ros.org/wiki/xacro">
     <xacro:property name="handle_mesh_file" value="handle_edited.obj"/>
-    <xacro:property name="handle_pos_x" value="0.0"/>
-    <xacro:property name="handle_pos_y" value="0.3"/>
-    <xacro:property name="handle_pos_z" value="0.0"/>
-    <xacro:property name="handle_ori_r" value="0.0"/>
-    <xacro:property name="handle_ori_p" value="0.0"/>
-    <xacro:property name="handle_ori_y" value="0.0"/>
-    <xacro:macro name="door_handle" params="">
+    <xacro:arg name="handle_pos_x" default="0.0"/>
+    <xacro:arg name="handle_pos_y" default="0.0"/>
+    <xacro:arg name="handle_pos_z" default="0.0"/>
+    <xacro:arg name="handle_ori_r" default="0.0"/>
+    <xacro:arg name="handle_ori_p" default="0.0"/>
+    <xacro:arg name="handle_ori_y" default="0.0"/>
+    <xacro:macro name="door_handle" params="handle_pos_x handle_pos_y handle_pos_z handle_ori_r handle_ori_p handle_ori_y">
         <joint name="handle_door" type="fixed">
             <!-- Hier xyz für door zu handle offset -->

File: scripts/complete_door.xacro (robot description, xacro)
@@ -3,7 +3,14 @@
     <xacro:property name="plane_xacro" value="plane.xacro"/>
     <xacro:property name="handle_xacro" value="handle.xacro"/>
+    <xacro:property name="handle_pos_x" value="0.0"/>
+    <xacro:property name="handle_pos_y" value="0.3"/>
+    <xacro:property name="handle_pos_z" value="0.0"/>
+    <xacro:property name="handle_ori_r" value="0.0"/>
+    <xacro:property name="handle_ori_p" value="0.0"/>
+    <xacro:property name="handle_ori_y" value="0.0"/>
     <xacro:include filename="plane.xacro"/>
     <xacro:door_plane parent="world"/>
     <xacro:include filename="handle.xacro"/>
-    <xacro:door_handle/>
+    <xacro:door_handle handle_pos_x="${handle_pos_x}" handle_pos_y="${handle_pos_y}"
+    handle_pos_z="${handle_pos_z}" handle_ori_r="${handle_ori_r}" handle_ori_p="${handle_ori_p}" handle_ori_y="${handle_ori_y}"/>
 </robot>

Commit message: handle template scale added

File: data/objs/pieces/handles/handle.xacro (robot description, xacro)
@@ -1,13 +1,4 @@
 <?xml version="1.0" encoding="utf-8"?>
 <robot name="door_handle" xmlns:xacro="http://www.ros.org/wiki/xacro">
-    <!--
-    <xacro:property name="handle_mesh_file" value="handle_edited.obj"/>
-    <xacro:arg name="handle_pos_x" default="0.0"/>
-    <xacro:arg name="handle_pos_y" default="0.0"/>
-    <xacro:arg name="handle_pos_z" default="0.0"/>
-    <xacro:arg name="handle_ori_r" default="0.0"/>
-    <xacro:arg name="handle_ori_p" default="0.0"/>
-    <xacro:arg name="handle_ori_y" default="0.0"/>
-    -->
     <xacro:macro name="door_handle" params="handle_pos_x handle_pos_y handle_pos_z handle_ori_r handle_ori_p handle_ori_y">
         <joint name="handle_door" type="fixed">
@@ -23,5 +14,5 @@
                 <origin xyz="0 0 0" />
                 <geometry>
-                    <mesh filename="${handle_mesh_file}" rpy="0 0 0" />
+                    <mesh filename="${handle_mesh_file}" rpy="0 0 0" scale="1 1 1" />
                 </geometry>
             </visual>
@@ -29,5 +20,5 @@
                 <origin xyz="0 0 0" />
                 <geometry>
-                    <mesh filename="${handle_mesh_file}" rpy="0 0 0" />
+                    <mesh filename="${handle_mesh_file}" rpy="0 0 0" scale="1 1 1" />
                 </geometry>
             </collision>
